Commit message: xacro file, move xacro file

File: urdf_tutorial/urdf/r2d2.urdf.xacro (robot description, xacro)
@@ -1,4 +1,15 @@
-<robot name="r2d2">
-<!-- base -->
+<?xml version="1.0" ?>
+<robot xmlns:xacro="http://ros.org/wiki/xacro" name="r2d2">
+<xacro:property name="base_width" value="0.2" />
+<xacro:property name="base_height" value="1.2" />
+<material name="white">
+    <color rgba="1 1 1 1"/>
+</material>
+<material name="grey">
+    <color rgba=".2 .2 .2 1" />
+</material>
+<material name="black">
+    <color rgba="0 0 0 1"/>
+</material>
 <link name="base">
   <visual>
@@ -7,7 +18,7 @@
       <cylinder radius="0.2" length="1.2" />
     </geometry>
+    <material name="grey"/>
   </visual>
 </link>
-<!-- arm1 -->
 <link name="arm1">
   <visual>
@@ -16,4 +27,5 @@
       <box size=".1 .18 1" />
     </geometry>
+    <material name="white"/>
   </visual>
 </link>
@@ -30,4 +42,5 @@
       <box size=".1 .15 0.6" />
     </geometry>
+    <material name="white"/>
   </visual>
 </link>
@@ -43,4 +56,5 @@
       <box size=".05 .1 0.3" />
     </geometry>
+    <material name="black"/>
   </visual>
 </link>
@@ -56,6 +70,8 @@
       <box size=".1 .05 .05" />
     </geometry>
+    <material name="grey"/>
   </visual>
 </link>
+<!-- co to? -->
 <joint name="end"  type="fixed">
   <origin rpy="0 0 0" xyz="0 0 0" />
@@ -63,29 +79,3 @@
   <child link="gripper"/>
 </joint>
-<link name="rod">
-  <!-- <visual>
-    <origin rpy="0 0 0" xyz="0.026 0 0.0" />
-    <geometry>
-      <box size=".05 .1 0.6" />
-    </geometry>
-  </visual> -->
-</link>
-<joint name="periscope"  type="fixed">
-  <!-- <origin xyz=".545 0 0.05" /> -->
-  <parent link="gripper"/>
-  <child link="rod"/>
-</joint>
-<link name="box">
-  <!-- <visual>
-    <origin rpy="0 0 0" xyz="0 0 0.025" />
-    <geometry>
-      <box size=".1 .05 .05" />
-    </geometry>
-  </visual> -->
-</link>
-<joint name="boxconnect" type="fixed">
-  <!-- <origin rpy="0 3.14 0" xyz="0.026 0 -0.3" /> -->
-  <parent link="rod"/>
-  <child link="box"/>
-</joint>
 </robot>

File: urdf_tutorial/urdf/r2d2_move.urdf.xacro (robot description, xacro)
@@ -1,4 +1,15 @@
-<robot name="r2d2">
-<!-- base -->
+<?xml version="1.0" ?>
+<robot xmlns:xacro="http://ros.org/wiki/xacro" name="r2d2">
+<xacro:property name="base_width" value="0.2" />
+<xacro:property name="base_height" value="1.2" />
+<material name="white">
+    <color rgba="1 1 1 1"/>
+</material>
+<material name="grey">
+    <color rgba=".2 .2 .2 1" />
+</material>
+<material name="black">
+    <color rgba="0 0 0 1"/>
+</material>
 <link name="base">
   <visual>
@@ -7,7 +18,7 @@
       <cylinder radius="0.2" length="1.2" />
     </geometry>
+    <material name="grey"/>
   </visual>
 </link>
-<!-- arm1 -->
 <link name="arm1">
   <visual>
@@ -16,7 +27,9 @@
       <box size=".1 .18 1" />
     </geometry>
+    <material name="white"/>
   </visual>
 </link>
-<joint name="arm1connect" type="fixed">
+<joint name="arm1connect" type="continuous">
+  <axis xyz="0 0 1"/>
   <origin xyz="0 0 1.2" />
   <parent link="base"/>
@@ -30,7 +43,9 @@
       <box size=".1 .15 0.6" />
     </geometry>
+    <material name="white"/>
   </visual>
 </link>
-<joint name="arm2connect" type="fixed">
+<joint name="arm2connect" type="continuous">
+  <axis xyz="0 0 1"/>
   <origin xyz="1 0 0" />
   <parent link="arm1"/>
@@ -43,7 +58,9 @@
       <box size=".05 .1 0.3" />
     </geometry>
+    <material name="black"/>
   </visual>
 </link>
-<joint name="wristconnect" type="fixed">
+<joint name="wristconnect" type="prismatic">
+  <limit effort="1000.0" lower="-0.2" upper="0" velocity="0.5"/>
   <origin rpy="0 3.14 0" xyz="0.6 0 0" />
   <parent link="arm2"/>
@@ -56,6 +73,8 @@
       <box size=".1 .05 .05" />
     </geometry>
+    <material name="grey"/>
   </visual>
 </link>
+<!-- co to? -->
 <joint name="end"  type="fixed">
   <origin rpy="0 0 0" xyz="0 0 0" />
@@ -63,29 +82,3 @@
   <child link="gripper"/>
 </joint>
-<link name="rod">
-  <!-- <visual>
-    <origin rpy="0 0 0" xyz="0.026 0 0.0" />
-    <geometry>
-      <box size=".05 .1 0.6" />
-    </geometry>
-  </visual> -->
-</link>
-<joint name="periscope"  type="fixed">
-  <!-- <origin xyz=".545 0 0.05" /> -->
-  <parent link="gripper"/>
-  <child link="rod"/>
-</joint>
-<link name="box">
-  <!-- <visual>
-    <origin rpy="0 0 0" xyz="0 0 0.025" />
-    <geometry>
-      <box size=".1 .05 .05" />
-    </geometry>
-  </visual> -->
-</link>
-<joint name="boxconnect" type="fixed">
-  <!-- <origin rpy="0 3.14 0" xyz="0.026 0 -0.3" /> -->
-  <parent link="rod"/>
-  <child link="box"/>
-</joint>
 </robot>
